File: Croaky4.sch (KiCad schematic (older format))
At the start: 31 parts, among them SW1 SW_Push, SW2 Rotary_Encoder_Switch, U1 PRTR5V0U2X, U2 ATmega32U2-AU, Y1 16MHz

Commit message: First prototype order
Parts:
- removed C5: 0.1uF, Capacitor_SMD:C_0805_2012Metric, symbol Device:C_Small
- removed R10, R7, R8, R9: 1k, Resistor_SMD:R_0805_2012Metric, symbol Device:R_Small
- added C10, C11, C12, C13, C7, C8, C9: .1uF, Capacitor_SMD:C_0805_2012Metric, symbol Device:C_Small
- added D4, D5, D6, D7: WS2812B, Keebio-Parts:WS2812B_flipped, symbol LED:WS2812B
- added J1: AVR-ISP-6, random-keyboard-parts:Reset_Pretty-Mask, symbol Connector:AVR-ISP-6
- C1, C2: LCSC (none) -> C112618
- C3, C4: LCSC (none) -> C393683
- C5: renamed from C6; value 10uF -> 4.7uF; LCSC (none) -> C162421
- C6: renamed from C7; LCSC (none) -> C126585
- F1: LCSC (none) -> C207149
- MX1, MX2, MX3, MX4: footprint MX_Only:MXOnly-1U -> MX_Only:MXOnly-1U-NoLED; symbol MX_Alps_Hybrid:MX-LED -> MX_Alps_Hybrid:MX-NoLED
- R1, R2: LCSC (none) -> C413697
- R3, R6: LCSC (none) -> C192906
- R4, R5: LCSC (none) -> C150390
- SW1: LCSC (none) -> C221929
- U1: renamed from U2; LCSC (none) -> C618733
- U2: renamed from U1; LCSC (none) -> C12333
- USB1: footprint Connector_USB:USB_C_Receptacle_HRO_TYPE-C-31-M-12 -> Keebio-Parts:HRO-TYPE-C-31-M-12-Assembly; LCSC (none) -> C165948
- Y1: LCSC (none) -> C254368
Connections:
- net ENCS2 is gone; now on net ROW0: MX1.2 (ROW), MX2.2 (ROW), MX3.2 (ROW), MX4.2 (ROW), SW2.S2
- net +5V: now also C10.2, C11.2, C12.2, C13.2, C7.2, C8.2, C9.2, D4.1 (VDD), D5.1 (VDD), D6.1 (VDD), D7.1 (VDD), J1.2 (VCC); no longer MX1.3 (LED), MX2.3 (LED), MX3.3 (LED), MX4.3 (LED)
- net COL0: now also U1.6 (PD0)
- net COL1: now also U1.7 (PD1)
- net COL2: now also U1.9 (PD3)
- net COL3: now also U1.8 (PD2)
- net COL4: now also U1.11 (PD5)
- net ENCA: now also U1.16 (PB2), J1.4 (MOSI)
- net ENCB: now also U1.15 (PB1), J1.3 (SCK)
- net GND: now also C10.1, C11.1, C12.1, C13.1, C7.1, C8.1, C9.1, D4.3 (VSS), D5.3 (VSS), D6.3 (VSS), D7.3 (VSS), J1.6 (GND)
- net RGBLED: now also U1.12 (PD6); no longer U1.9 (PD3)
- net RESET: now reaches R3.1, SW1.2, U1.24 (PC1/~RESET)
- net RESET: now also J1.5 (~RST)
- net ROW0: now reaches U1.10 (PD4)
- net MISO: now reaches U1.17 (PB3)
- net MISO: now also J1.1 (MISO)
- net at D3.2 (DOUT): now also D4.4 (DIN)
- new net: D4.2 (DOUT), D5.4 (DIN)
- new net: D5.2 (DOUT), D6.4 (DIN)
- new net: D6.2 (DOUT), D7.4 (DIN)
Other:
- moved on the sheet: C5, D1, D2, D3, R6, SW2
